Commit message: yjhrot

File: resources/robots/XBot/urdf/XBot-LNoArm.urdf (robot description, URDF)
Before this commit: robot XBot-L, 91 links, 90 joints
Joints:
- joint left_elbow_pitch_joint: type revolute -> fixed
- joint left_shoulder_pitch_joint: type revolute -> fixed
- joint left_wrist_roll_joint: type revolute -> fixed
- joint right_elbow_pitch_joint: type revolute -> fixed
- joint right_shoulder_pitch_joint: type revolute -> fixed
- joint right_wrist_roll_joint: type revolute -> fixed
